File: BarrelJackAdapter/BarrelJackAdapter.kicad_sch (KiCad schematic)
At the start: 6 parts, among them J1 Barrel_Jack_Switch, J2 Conn_01x03, J4 Conn_01x03, U1 L7805

Commit message: wip v2
Parts:
- removed J2, J4: Conn_01x03, Connector_PinHeader_2.54mm:PinHeader_1x03_P2.54mm_Vertical, symbol Connector_Generic:Conn_01x03
- removed U1: L7805, Package_TO_SOT_THT:TO-220-3_Vertical, symbol Regulator_Linear:L7805
- added C3: 10u, Capacitor_SMD:C_0201_0603Metric, symbol Device:C_Small
- added J2, J3, J4, J5: Conn_02x03_Counter_Clockwise, Connector_PinHeader_2.54mm:PinHeader_2x03_P2.54mm_Vertical, symbol Connector_Generic:Conn_02x03_Odd_Even
- added U1: LD1117S33TR_SOT223, Package_TO_SOT_SMD:SOT-223-3_TabPin2, symbol Regulator_Linear:LD1117S33TR_SOT223
- added U2: L7805, Package_TO_SOT_SMD:TO-263-2, symbol Regulator_Linear:L7805
Connections:
- net +5V: now also J3.6 (Pin_6), J5.6 (Pin_6), U1.3 (VI), U2.3 (OUT)
- net +9V: now also J3.2 (Pin_2), J5.2 (Pin_2), U2.1 (IN)
- net GND: now also C3.2, J2.2 (Pin_2), J2.4 (Pin_4), J2.6 (Pin_6), J4.2 (Pin_2), J4.4 (Pin_4), J4.6 (Pin_6), U1.1 (GND), U2.2 (GND)
- new net +3.3V: C3.1, J3.3 (Pin_3), J5.3 (Pin_3), U1.2 (VO)
- new net Vleft: J2.1 (Pin_1), J2.3 (Pin_3), J2.5 (Pin_5), J3.4 (Pin_4)
- new net Vright: J4.1 (Pin_1), J4.3 (Pin_3), J4.5 (Pin_5), J5.4 (Pin_4)
- no-connect marks 0 -> 4
Other:
- note added: "1.7 in between inner rails here (Breadboard rail spacing)."
- moved on the sheet: C1, C2, J1
